Commit message: debug

File: slamkit2d_description/urdf/slamkit2d_urdf.xacro (robot description, xacro)
@@ -1,5 +1,20 @@
 <?xml version="1.0"?>
 <robot name="slamkit2d_urdf" xmlns:xacro="http://www.ros.org/wiki/xacro">
-  <xacro:include filename="$(find neobot_description)/urdf/neobot_essential.xacro" />
+  <!-- Defining the colors used in this robot -->
+  <material name="Black">
+    <color rgba="0.0 0.0 0.0 1.0"/>
+  </material>
+  <material name="White">
+    <color rgba="1.0 1.0 1.0 1.0"/>
+  </material>
+  <material name="Red">
+    <color rgba="0.8 0.0 0.0 1.0"/>
+  </material>
+  <material name="Green">
+    <color rgba="0.0 0.8 0.0 1.0"/>
+  </material>
+  <material name="Blue">
+    <color rgba="0.0 0.0 0.8 1.0"/>
+  </material>
   <!-- <link name="base_footprint"/> -->
   <!-- base_link --> <!--Actual body-->
